File: Keyboard-USB-Hub.kicad_pcb (KiCad board)
At the start: 4 copper layers, 78 x 24 mm, 57 parts, among them J1 USB_Internal, J2 I2C, J3 USB_A, J4 USB_A, J5 USB_C_Receptacle_USB2.0_16P, Q1 PMOS, Q2 PMOS, Q3 PMOS, U1 LDL212PV33R, U2 24LC04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

Commit message: Add LED
Parts:
- added D2: LED, LED_SMD:LED_0603_1608Metric, F.Cu at (149.9, 121.0)
- added R18: 1k, Resistor_SMD:R_0402_1005Metric, F.Cu at (149.8, 119.5)
Connections:
- J1 pad MP: GND -> (no net)
- J2 pad MP: GND -> (no net)
- J3 pad MP: GND -> (no net)
- J4 pad MP: GND -> (no net)
Routing:
- net +3V3: track 65.1 -> 77.3 mm, vias 11 -> 12
- net Net-(D2-K): track 0.00 -> 1.58 mm
- net GND: vias 77 -> 79
