File: Keyboard-USB-Hub.kicad_sch (KiCad schematic)
At the start: 55 parts, among them J1 USB_Internal, J2 I2C, J3 USB_A, J4 USB_A, J5 USB_C_Receptacle_USB2.0_16P, Q1 PMOS, Q2 PMOS, Q3 PMOS, U1 LDL212PV33R, U2 24LC04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

Commit message: Add LED
Parts:
- added D2: LED, LED_SMD:LED_0603_1608Metric, symbol Device:LED
- added R18: 1k, Resistor_SMD:R_0402_1005Metric, symbol Device:R
Connections:
- net +3V3: now also D2.2 (A)
- net GND: now also R18.2
- new net: D2.1 (K), R18.1
